Commit message: Port verified FEM ground pick to native Jazzy
Add reproducible English and Traditional Chinese Jazzy runbooks, source-based bootstrap scripts, direct-start configuration, and verified FEM lift/release records.

File: urdf/ur5_robotiq.urdf.xacro (robot description, xacro)
@@ -21,4 +21,8 @@
   <xacro:arg name="safety_k_position" default="20"/>
   <xacro:arg name="use_fake_hardware" default="true"/>
+  <xacro:arg
+    name="initial_positions_file"
+    default="$(find ur5_moveit_demo)/config/jazzy_fem_initial_positions.yaml"/>
+  <xacro:property name="initial_positions_file" default="$(arg initial_positions_file)"/>
   <xacro:arg name="script_filename" default="ros_control.urscript"/>
   <xacro:arg name="input_recipe_filename" default="rtde_input_recipe.txt"/>
@@ -47,5 +51,6 @@
     name="$(arg name)"
     tf_prefix="$(arg prefix)"
-    mock_sensor_commands="false"/>
+    mock_sensor_commands="false"
+    initial_positions="${xacro.load_yaml(initial_positions_file)}"/>
   <xacro:ur_to_robotiq
     prefix=""
